File: KiCad/InclinationMeter.kicad_pcb (KiCad board)
At the start: 4 copper layers, 130 x 35 mm, 48 parts, among them J1 FTSH-107-01-L-DV-K, J2 FH12-10S-0.5SH, Q1 DMG2305UX, Q2 FS8205A, U1 DW01A, U10 LM35DGS, U2 TP4056, U3 LP5907MFX-3.3, U4 SD6210A, U5 RN4871-I_RM128, U6 STM32G0B1RET6, U7 SN74AHCT244DBR, U8 SN74HC14PWR, U9 24LC256-I_ST, Y1 8MHz

Commit message: Schematic finalized
Parts:
- removed J2: FH12-10S-0.5SH, local_FH12-10S:FPC-SMD_FH12-10S-0.5SH-55
- added C23: 100n, sldrnrd:C_0603, F.Cu at (86.7, 79.8)
- added C24: 10n, sldrnrd:C_0603, F.Cu at (65.1, 34.3)
- added C25: 10n, sldrnrd:C_0603, F.Cu at (65.1, 36.8)
- added C26: 100n, sldrnrd:C_0603, F.Cu at (65.1, 39.3)
- added C27: 100n, sldrnrd:C_0603, F.Cu at (65.1, 41.8)
- added C28: 100n, sldrnrd:C_0603, F.Cu at (65.1, 44.3)
- added C29: 3u3, sldrnrd:C_0805, F.Cu at (70.2, 62.3)
- added C30: 100n, sldrnrd:C_0603, F.Cu at (65.1, 46.8)
- added C31: 10n, sldrnrd:C_0603, F.Cu at (65.1, 49.3)
- added C32: 100n, sldrnrd:C_0603, F.Cu at (69.1, 34.3)
- added C33: 10n, sldrnrd:C_0603, F.Cu at (69.1, 36.8)
- added C34: 100n, sldrnrd:C_0603, F.Cu at (69.1, 39.3)
- added C35: 100n, sldrnrd:C_0603, F.Cu at (69.1, 41.8)
- added C36: 100n, sldrnrd:C_0603, F.Cu at (69.1, 44.3)
- added C37: 100n, sldrnrd:C_0603, F.Cu at (50.0, 71.3)
- added C38: 100n, sldrnrd:C_0603, F.Cu at (50.0, 73.8)
- added D3: BAT54WS, sldrnrd:SOD-323, F.Cu at (98.9, 40.4)
- added D4: BAT54WS, sldrnrd:SOD-323, F.Cu at (98.9, 43.3)
- added D5: LED_Red_0603, sldrnrd:LED_0603, F.Cu at (103.4, 55.0)
- added D6: LED_Green_0603, sldrnrd:LED_0603, F.Cu at (103.4, 57.6)
- added D7: LED_Green_0603, sldrnrd:LED_0603, F.Cu at (61.0, 60.4)
- added D8: LED_Green_0603, sldrnrd:LED_0603, F.Cu at (61.0, 63.0)
- added J3: Header_FFC_1.0mm_06, sldrnrd:Header_FFC_1.0mm_06, F.Cu at (58.9, 91.1)
- added J4: Header_50mil_2x07, sldrnrd:Header_50mil_2x07, F.Cu at (70.9, 91.4)
- added J5: Header_FFC_1.0mm_10, sldrnrd:Header_FFC_1.0mm_10, F.Cu at (60.9, 73.5)
- added J6: Header_FFC_1.0mm_10, sldrnrd:Header_FFC_1.0mm_10, F.Cu at (60.9, 82.3)
- added Q3: AO3400A, sldrnrd:SOT-23, F.Cu at (103.8, 47.0)
- added Q4: AO3400A, sldrnrd:SOT-23, F.Cu at (103.8, 51.5)
- added R10: 68k, sldrnrd:R_0603, F.Cu at (94.7, 49.3)
- added R11: 1k, sldrnrd:R_0603, F.Cu at (69.1, 46.8)
- added R12: 1k, sldrnrd:R_0603, F.Cu at (69.1, 49.3)
- added R13: 68k, sldrnrd:R_0603, F.Cu at (73.1, 34.3)
- added R14: 68k, sldrnrd:R_0603, F.Cu at (73.1, 36.8)
- added R15: 33k, sldrnrd:R_0603, F.Cu at (73.1, 39.3)
- added R16: 33k, sldrnrd:R_0603, F.Cu at (73.1, 41.8)
- added R17: 33k, sldrnrd:R_0603, F.Cu at (73.1, 44.3)
- added R18: 68k, sldrnrd:R_0603, F.Cu at (73.1, 46.8)
- added R19: 68k, sldrnrd:R_0603, F.Cu at (73.1, 49.3)
- added R20: 68k, sldrnrd:R_0603, F.Cu at (77.1, 34.3)
- added R21: 33k, sldrnrd:R_0603, F.Cu at (77.1, 36.8)
- added R22: 33k, sldrnrd:R_0603, F.Cu at (77.1, 39.3)
- added R23: 33k, sldrnrd:R_0603, F.Cu at (77.1, 41.8)
- added R24: 68k, sldrnrd:R_0603, F.Cu at (77.1, 44.3)
- added R25: 1k, sldrnrd:R_0603, F.Cu at (77.1, 46.8)
- added R26: 5k1, sldrnrd:R_0603, F.Cu at (50.0, 76.3)
- added R27: 100k, sldrnrd:R_0603, F.Cu at (50.0, 78.8)
- added R28: 5k1, sldrnrd:R_0603, F.Cu at (50.0, 81.3)
- added R29: 68k, sldrnrd:R_0603, F.Cu at (50.0, 83.8)
- added R30: 100k, sldrnrd:R_0603, F.Cu at (50.0, 86.3)
- added R31: 33k, sldrnrd:R_0603, F.Cu at (50.0, 88.8)
- added R9: 100k, sldrnrd:R_0603, F.Cu at (94.7, 46.8)
- added SW1: PEC11R-4215F-S0024, sldrnrd:RotaryEncoder_PEC11R, F.Cu at (140.0, 48.5)
- added SW2: PEC11R-4215F-S0024, sldrnrd:RotaryEncoder_PEC11R, F.Cu at (140.0, 68.0)
- added U11: LM35DGS, sldrnrd:SOT-23, F.Cu at (65.5, 63.0)
- added Y2: 8MHz, sldrnrd:CRYSTAL-3225, F.Cu at (104.2, 80.4)
- BZ1: footprint local_CPT-9019A:BUZ-SMD_L9.0-W9.0_CPT-9019A-SMT-TR -> sldrnrd:CPT-9019A
- C1: value 10uF -> 100n; footprint Capacitor_SMD:C_0603_1608Metric -> sldrnrd:C_0603
- C10, C17, C7: value 100nF -> 1uF; footprint Capacitor_SMD:C_0603_1608Metric -> sldrnrd:C_0603
- C11: value 33pF -> 10u; footprint Capacitor_SMD:C_0603_1608Metric -> sldrnrd:C_0805
- C12, C4: value 100nF -> 100n; footprint Capacitor_SMD:C_0603_1608Metric -> sldrnrd:C_0603
- C13: value 4.7uF -> 100n; footprint Capacitor_SMD:C_0805_2012Metric -> sldrnrd:C_0603
- C14, C18, C3: value 1uF -> 100n; footprint Capacitor_SMD:C_0603_1608Metric -> sldrnrd:C_0603
- C15: value 10nF -> 10u; footprint Capacitor_SMD:C_0603_1608Metric -> sldrnrd:C_0805
- C16: value 100nF -> 3u3; footprint Capacitor_SMD:C_0603_1608Metric -> sldrnrd:C_0805
- C19: value 1uF -> 12.5p; footprint Capacitor_SMD:C_0603_1608Metric -> sldrnrd:C_0603
- C2, C5: value 10uF -> 1uF; footprint Capacitor_SMD:C_0603_1608Metric -> sldrnrd:C_0603
- C20: value 100nF -> 12.5p; footprint Capacitor_SMD:C_0603_1608Metric -> sldrnrd:C_0603
- C21: value 100nF -> 20p; footprint Capacitor_SMD:C_0603_1608Metric -> sldrnrd:C_0603
- C22: value 10nF -> 20p; footprint Capacitor_SMD:C_0603_1608Metric -> sldrnrd:C_0603
- C6: value 1uF -> 10u; footprint Capacitor_SMD:C_0603_1608Metric -> sldrnrd:C_0603
- C8: value 10uF -> 10u; footprint Capacitor_SMD:C_0805_2012Metric -> sldrnrd:C_0603
- C9: value 33pF -> 100n; footprint Capacitor_SMD:C_0603_1608Metric -> sldrnrd:C_0603
- D1: value Green -> BAT54WS; footprint LED_SMD:LED_0603_1608Metric -> sldrnrd:SOD-323
- D2: value Blue -> BAT54WS; footprint LED_SMD:LED_0603_1608Metric -> sldrnrd:SOD-323
- J1: value FTSH-107-01-L-DV-K -> JST_PH_2.0mm_1x02; footprint local_FTSH-107:HDR-SMD_14P-P1.27_FTSH-107-01-L-DV-K -> sldrnrd:JST_PH_2.0mm_1x02
- Q1: footprint local_DMG2305UX:SOT-23-3_L2.9-W1.3-P1.90-LS2.4-BR -> sldrnrd:SOT-23-BR
- Q2: footprint local_FS8205A:TSSOP-8_L4.4-W3.0-P0.65-LS6.4-BL-2 -> sldrnrd:TSSOP-8
- R1: footprint Resistor_SMD:R_0603_1608Metric -> sldrnrd:R_0603
- R2: value 1k -> 10k; footprint Resistor_SMD:R_0603_1608Metric -> sldrnrd:R_0603
- R3: value 2.4k -> 2k; footprint Resistor_SMD:R_0603_1608Metric -> sldrnrd:R_0603
- R4: value 100k -> 1k; footprint Resistor_SMD:R_0603_1608Metric -> sldrnrd:R_0603
- R5: value 390k -> 2k; footprint Resistor_SMD:R_0603_1608Metric -> sldrnrd:R_0603
- R6: value 330R -> 33k; footprint Resistor_SMD:R_0603_1608Metric -> sldrnrd:R_0603
- R7: value 100R -> 1k; footprint Resistor_SMD:R_0603_1608Metric -> sldrnrd:R_0603
- R8: value 330R -> 1k; footprint Resistor_SMD:R_0603_1608Metric -> sldrnrd:R_0603
- U1: footprint local_DW01A:SOT-23-6_L2.9-W1.6-P0.95-LS2.8-BL -> sldrnrd:SOT-23-6
- U10: value LM35DGS -> SN74HC14PWR; footprint Package_TO_SOT_SMD:SOT-23 -> sldrnrd:TSSOP-14
- U2: value TP4056 -> LP5907MFX-3.3/NOPB; footprint local_TP4056:ESOP-8_L4.9-W3.9-P1.27-LS6.0-BL-EP -> sldrnrd:SOT-23-5
- U3: value LP5907MFX-3.3 -> TP4056; footprint local_LP5907:SOT-23-5_L3.0-W1.7-P0.95-LS2.8-BR -> sldrnrd:ESOP-8
- U4: value SD6210A -> LP5907MFX-3.3/NOPB; footprint local_SD6210A:SOT-23-6_L2.9-W1.6-P0.95-LS2.8-BL -> sldrnrd:SOT-23-5
- U5: value RN4871-I_RM128 -> SD6210A; footprint local_RN4871:BULETM-SMD_RN4871-V-RM118 -> sldrnrd:SOT-23-6
- U6: footprint Package_QFP:LQFP-64_10x10mm_P0.5mm -> sldrnrd:LQFP-64
- U7: value SN74AHCT244DBR -> RN4871-I_RM128; footprint local_SN74AHCT244DBR:SSOP-20_L7.2-W5.3-P0.65-LS7.8-BL -> sldrnrd:RN4871
- U8: value SN74HC14PWR -> SN74AHCT244DBR; footprint local_SN74HC14:TSSOP-14_L5.0-W4.4-P0.65-LS6.4-BL -> sldrnrd:SSOP-20
- U9: footprint local_24LC256:TSSOP-8_L4.4-W3.0-P0.65-LS6.4-BL -> sldrnrd:TSSOP-8
- Y1: value 8MHz -> 32.768kHz; footprint local_X50328MSB2GI:CRYSTAL-SMD_L5.0-W3.2 -> sldrnrd:CRYSTAL-3215
- moved Q1 80.3 mm to (107.5, 55.8)
- moved U10 73.6 mm to (55.8, 63.2)
- moved J1 68.0 mm to (107.0, 34.5)
- moved R5 67.8 mm to (94.7, 36.8)
- moved R4 67.1 mm to (94.7, 34.3)
- moved BZ1 61.5 mm to (68.5, 55.7)
- moved R1 60.9 mm to (90.7, 46.8)
- moved U5 58.7 mm to (108.7, 51.4)
- moved U3 57.6 mm to (93.2, 57.1)
- moved Y1 56.8 mm to (103.2, 84.5)
- moved R2 56.2 mm to (90.7, 49.3)
- moved C6 52.7 mm to (86.7, 46.8)
- moved U4 52.5 mm to (87.0, 59.4)
- moved C18 52.0 mm to (86.7, 67.2)
- moved C2 52.0 mm to (86.7, 36.8)
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Connections:
- net /Power Supply/PROT_OC renamed Net-(Q2-G2)
- net /Power Supply/PROT_OD renamed Net-(Q2-G1)
- net USB_DM renamed USB_D-
- net USB_DP renamed USB_D+
- BZ1 pad 1: BUZZER -> BUZZER_5V
- BZ1 pad 2: OSC_IN -> GND
- C1 pad 1: OSC_IN -> LDO_EN
- C1 pad 2: OSC_IN -> GND
- C10 pad 1: GND -> 3V3_Sensors
- C10 pad 2: OSC_IN -> GND
- C11 pad 1: OSC_OUT -> 5V0
- C11 pad 2: OSC_IN -> GND
- C12 pad 1: GND -> 5V0
- C12 pad 2: OSC_IN -> GND
- C13 pad 1: GND -> VCC
- C13 pad 2: OSC_IN -> GND
- C14 pad 1: GND -> BATTERY_SENSE
- C14 pad 2: OSC_IN -> GND
- C15 pad 1: GND -> VCC
- C15 pad 2: OSC_IN -> GND
- C16 pad 1: GND -> Net-(U5-C+)
- C16 pad 2: OSC_IN -> Net-(U5-C-)
- C17 pad 1: OSC_IN -> VCC
- C17 pad 2: OSC_IN -> GND
- C18 pad 1: OSC_IN -> VCC
- C18 pad 2: OSC_IN -> GND
- C19 pad 1: OSC_IN -> Net-(U6-PC14)
- C19 pad 2: OSC_IN -> GND
- C2 pad 1: +5V -> VCC
- C2 pad 2: OSC_IN -> GND
- C20 pad 1: GND -> Net-(U6-PC15)
- C20 pad 2: OSC_IN -> GND
- C21 pad 1: GND -> Net-(U6-PF0)
- C21 pad 2: OSC_IN -> GND
- C22 pad 1: GND -> Net-(U6-PF1)
- C22 pad 2: OSC_IN -> GND
- C3 pad 1: VBAT -> Net-(U1-VCC)
- C3 pad 2: OSC_IN -> BAT-
- C4 pad 1: OSC_IN -> 3V3
- C4 pad 2: OSC_IN -> GND
- C5 pad 1: OSC_IN -> 3V3
- C5 pad 2: OSC_IN -> GND
- C6 pad 1: VBAT -> V_USB
- C6 pad 2: /Power Supply/CFLY_N -> GND
- C7 pad 1: GND -> VCC
- C7 pad 2: OSC_IN -> GND
- C8 pad 1: GND -> VCC
- C8 pad 2: OSC_IN -> GND
- C9 pad 1: OSC_IN -> 3V3_Sensors
- C9 pad 2: OSC_IN -> GND
- D1 pad 1: Net-(D1-A) -> Net-(D1-K)
- D1 pad 2: OSC_IN -> V_USB
- D2 pad 1: Net-(D2-A) -> Net-(D1-K)
- D2 pad 2: OSC_IN -> PWR_ON
- Q1 pad 2: VBAT_RAW -> VCC
- Q1 pad 3: VBAT -> BAT+
- Q2 pad 2: CELL_NEG -> BAT-
- Q2 pad 3: CELL_NEG -> BAT-
- Q2 pad 6: OSC_IN -> GND
- Q2 pad 7: OSC_IN -> GND
- R1 pad 1: OSC_IN -> BAT-
- R2 pad 1: OSC_IN -> Net-(D1-K)
- R2 pad 2: Net-(U1-CSI) -> LDO_EN
- R3 pad 1: OSC_IN -> Net-(U1-CS)
- R3 pad 2: OSC_IN -> GND
- R4 pad 1: VBAT -> Net-(U1-VCC)
- R4 pad 2: VBAT_SENSE -> VCC
- R5 pad 1: VBAT_SENSE -> GND
- R5 pad 2: OSC_IN -> Net-(U3-PROG)
- R6 pad 1: LED_PWR -> V_USB
- R6 pad 2: Net-(D1-A) -> Net-(Q3-D)
- R7 pad 1: Net-(U10-VOUT) -> 3V3
- R7 pad 2: TEMP_SENSE -> Net-(D5-A)
- R8 pad 1: LED_STS -> 3V3
- R8 pad 2: Net-(D2-A) -> Net-(D6-A)
- U1 pad 2: Net-(U1-CSI) -> Net-(U1-CS)
- U1 pad 5: /Power Supply/DW01_VDD -> Net-(U1-VCC)
- U1 pad 6: CELL_NEG -> BAT-
- U10 pad 1: GND -> ~{ENC_1A_RAW}
- U10 pad 2: Net-(U10-VOUT) -> ENC_1A
- U10 pad 3: OSC_IN -> ~{ENC_1B_RAW}
- U2 pad 1: OSC_IN -> VCC
- U2 pad 2: OSC_IN -> GND
- U2 pad 3: OSC_IN -> LDO_EN
- U2 pad 4: OSC_IN -> unconnected-(U2-N/C-Pad4)
- U2 pad 5: VBAT -> 3V3
- U3 pad 1: VBAT -> GND
- U3 pad 2: OSC_IN -> Net-(U3-PROG)
- U3 pad 3: OSC_IN -> GND
- U3 pad 4: unconnected-(U3-N/C-Pad4) -> V_USB
- U3 pad 5: OSC_IN -> VCC
- U4 pad 1: +5V -> VCC
- U4 pad 2: OSC_IN -> GND
- U4 pad 3: OSC_IN -> LDO_EN
- U4 pad 4: /Power Supply/CFLY_N -> unconnected-(U4-N/C-Pad4)
- U4 pad 5: VBAT -> 3V3_Sensors
- U5 pad 1: unconnected-(U5-NC-Pad1) -> 5V0
- U5 pad 2: OSC_IN -> GND
- U5 pad 3: OSC_IN -> 5V_EN
- U5 pad 4: unconnected-(U5-P1_3-Pad4) -> Net-(U5-C-)
- U5 pad 5: unconnected-(U5-P1_7-Pad5) -> VCC
- U5 pad 6: unconnected-(U5-P1_6-Pad6) -> Net-(U5-C+)
- U6 pad 1: unconnected-(U6-PC11-Pad1) -> ENC_2B
- U6 pad 10: OSC_IN -> Net-(U6-PF0)
- U6 pad 11: OSC_OUT -> Net-(U6-PF1)
- U6 pad 12: NRST -> ~{RST}
- U6 pad 13: GND -> PCAP04_2_SCL
- U6 pad 14: LED_PWR -> PCAP04_2_SDA
- U6 pad 15: LED_STS -> PCAP04_2_P3
- U6 pad 16: unconnected-(U6-PC3-Pad16) -> PCAP04_2_P2
- U6 pad 17: ENC1_A -> PCAP04_2_INT
- U6 pad 18: ENC1_B -> 3V3_EN
- U6 pad 19: ENC1_SW -> 5V_EN
- U6 pad 2: unconnected-(U6-PC12-Pad2) -> ENC_2A
- U6 pad 20: ENC2_A -> ~{CHARGE_EN}
- U6 pad 21: DISP_CS -> SCL3300_CS
- U6 pad 22: DISP_SCK -> SCL3300_SCK
- U6 pad 23: DISP_VCOM -> SCL3300_MISO
- U6 pad 24: DISP_MOSI -> SCL3300_MOSI
- U6 pad 25: ENC2_B -> BLE_UART_MCU_TO_BLE
- U6 pad 26: ENC2_SW -> BLE_UART_BLE_TO_MCU
- U6 pad 27: VBAT_SENSE -> ~{BLE_RST}
- U6 pad 28: TEMP_SENSE -> BLE_P1_6
- U6 pad 29: unconnected-(U6-PB2-Pad29) -> BLE_P0_2
- U6 pad 3: unconnected-(U6-PC13-Pad3) -> ENC_2SW
- U6 pad 30: I2C2_SCL -> BLE_P3_6
- U6 pad 31: I2C2_SDA -> BLE_P1_7
- U6 pad 32: SCL_CS -> BLE_P2_0
- U6 pad 33: SPI2_SCK -> PCAP04_1_SCL
- U6 pad 34: SPI2_MISO -> PCAP04_1_SDA
- U6 pad 35: SPI2_MOSI -> PCAP04_1_P2
- U6 pad 36: DISP_ON -> PCAP04_1_P3
- U6 pad 37: CHG_SENSE -> PCAP04_1_INT
- U6 pad 38: PCAP1_INT -> unconnected-(U6-PC6-Pad38)
- U6 pad 39: PCAP2_INT -> unconnected-(U6-PC7-Pad39)
- U6 pad 4: unconnected-(U6-PC14/OSC32_IN-Pad4) -> Net-(U6-PC14)
- U6 pad 40: unconnected-(U6-PD8-Pad40) -> DEBUG_UART_MCU_TO_PC
- U6 pad 41: unconnected-(U6-PD9-Pad41) -> DEBUG_UART_PC_TO_MCU
- U6 pad 47: BLE_RST -> BATTERY_SENSE
- U6 pad 48: BLE_STATUS -> TEMP_SENSE
- U6 pad 49: PCAP1_RST -> BUZZER
- U6 pad 5: GND -> Net-(U6-PC15)
- U6 pad 50: PCAP2_RST -> DISP_CS
- U6 pad 51: unconnected-(U6-PD1-Pad51) -> DISP_SCK
- U6 pad 52: unconnected-(U6-PD2-Pad52) -> DISP_ON
- U6 pad 53: unconnected-(U6-PD3-Pad53) -> DISP_VCOM
- U6 pad 54: unconnected-(U6-PD4-Pad54) -> DISP_MOSI
- U6 pad 55: unconnected-(U6-PD5-Pad55) -> STANDBY_SENSE
- U6 pad 56: unconnected-(U6-PD6-Pad56) -> CHARGE_SENSE
- U6 pad 57: BUZZER -> SWO
- U6 pad 58: unconnected-(U6-PB4-Pad58) -> LED_PWR
- U6 pad 59: unconnected-(U6-PB5-Pad59) -> LED_STATUS
- U6 pad 6: GND -> unconnected-(U6-VBAT-Pad6)
- U6 pad 60: BLE_TX -> EEPROM_SCL
- U6 pad 61: BLE_RX -> EEPROM_SDA
- U6 pad 62: I2C1_SCL -> ENC_1B
- U6 pad 63: I2C1_SDA -> ENC_1A
- U6 pad 64: unconnected-(U6-PC10-Pad64) -> ~{ENC_1SW}
- U6 pad 8: GND -> VCC
- U6 pad 9: OSC_IN -> GND
- U7 pad 1: OSC_IN -> unconnected-(U7-NC-Pad1)
- U7 pad 10: OSC_IN -> ~{BLE_RST}
- U7 pad 11: DISP_ON -> unconnected-(U7-P0_0-Pad11)
- U7 pad 12: /Display/DISP_VCOM_5V -> BLE_P0_2
- U7 pad 13: unconnected-(U7-2A2-Pad13) -> GND
- U7 pad 14: /Display/DISP_CS_5V -> VCC
- U7 pad 16: /Display/DISP_MOSI_5V -> BLE_P2_0
- U7 pad 2: OSC_IN -> GND
- U7 pad 3: OSC_IN -> unconnected-(U7-P1_2-Pad3)
- U7 pad 4: OSC_IN -> unconnected-(U7-P1_3-Pad4)
- U7 pad 5: OSC_IN -> BLE_P1_7
- U7 pad 6: OSC_IN -> BLE_P1_6
- U7 pad 7: OSC_IN -> BLE_UART_MCU_TO_BLE
- U7 pad 8: OSC_IN -> BLE_UART_BLE_TO_MCU
- U7 pad 9: OSC_IN -> BLE_P3_6
- U8 pad 1: ENC1_A -> GND
- U8 pad 10: ENC2_B -> unconnected-(U8-GND-Pad10)
- U8 pad 11: /UI & Peripherals/ENC2_B_RAW -> BUZZER
- U8 pad 12: ENC2_SW -> DISP_VCOM_5V
- U8 pad 13: /UI & Peripherals/ENC2_SW_RAW -> BUZZER
- U8 pad 14: GND -> DISP_CS_5V
- U8 pad 2: ENC1_A -> DISP_SCK
- U8 pad 3: /UI & Peripherals/ENC1_B_RAW -> DISP_ON_5V
- U8 pad 4: ENC1_B -> DISP_MOSI
- U8 pad 5: /UI & Peripherals/ENC1_SW_RAW -> BUZZER_5V
- U8 pad 6: ENC1_SW -> DISP_CS
- U8 pad 7: OSC_IN -> BUZZER_5V
- U8 pad 8: ENC2_A -> DISP_VCOM
- U8 pad 9: /UI & Peripherals/ENC2_A_RAW -> BUZZER_5V
- U9 pad 1: OSC_IN -> GND
- U9 pad 2: OSC_IN -> GND
- U9 pad 3: OSC_IN -> GND
- U9 pad 4: OSC_IN -> GND
- U9 pad 5: I2C1_SDA -> EEPROM_SDA
- U9 pad 6: I2C1_SCL -> EEPROM_SCL
- U9 pad 7: OSC_IN -> GND
- U9 pad 8: GND -> 3V3
- Y1 pad 1: OSC_IN -> Net-(U6-PC15)
- Y1 pad 2: OSC_OUT -> Net-(U6-PC14)
