File: KiCad/mcu.kicad_sch (KiCad schematic)
At the start: 10 parts, among them U1 STM32G0B1RET6, Y1 8MHz

Commit message: Schematics edited manually
Parts:
- added C18, C21: 100nF, sldrnrd:C_0603, symbol sldrnrd:Capacitor/C_0603
- added C19: 10uF, sldrnrd:C_0805, symbol sldrnrd:Capacitor/C_0805
- added C22: 10nF, sldrnrd:C_0603, symbol sldrnrd:Capacitor/C_0603
- added J2: USB-C, sldrnrd:USB_C, symbol sldrnrd:Connector/USB/USB_C
- added J3: FTSH-107-01-L-DV-K, sldrnrd:HDR-SMD_14P-P1.27_FTSH-107-01-L-DV-K, symbol sldrnrd:Connector/50Mil/Header_50mil_2x07
- added R8: 100R, sldrnrd:R_0603, symbol sldrnrd:Resistor/R_0603
- added U11: LM35DGS, sldrnrd:SOT-23, symbol sldrnrd:Sensor/LM35
- added U2: RN4871-I_RM128, sldrnrd:RN4871, symbol sldrnrd:Wireless/Bluetooth/RN4871-I_RM128
- added U9: 24LC256-I_ST, sldrnrd:TSSOP-8, symbol sldrnrd:Memory/EEPROM/24LC256-I_ST
Connections:
- net +3V3: now also C9.1, C18.1, C19.1, C21.1, C22.1, J3.01 (1), U11.1 (VS+), U2.14 (VBAT), U2.15 (P2_7), U2.16 (P2_0), U9.8 (VCC)
- net BLE_RST: now also U2.10 (RST_N)
- net BLE_RX: now also U2.8 (UART_TX)
- net BLE_STATUS: now also U2.11 (P0_0)
- net BLE_TX: now also U2.7 (UART_RX)
- net GND: now also C9.2, C18.2, C19.2, C21.2, C22.2, J3.03 (3), J3.05 (5), J3.07 (7), J3.09 (9), J3.11, J3.13, J3.14, U11.3 (GND), U2.12 (P0_2), U2.13 (GND), U2.2 (GND), U2.3 (P1_2), U9.1 (A0), U9.2 (A1), U9.3 (A2), U9.4 (VSS), U9.7 (WP)
- net I2C1_SCL: now also U9.6 (SCL)
- net I2C1_SDA: now also U9.5 (SDA)
- net NRST: now also J3.10
- net SWCLK: now also J3.04 (4)
- net SWDIO: now also J3.02 (2)
- net TEMP_SENSE: now also R8.2
- new net: R8.1, U11.2 (VOUT)
- no-connect marks 0 -> 13
Other:
- note added: "100R series on SWDIO/SWCLK"
- note added: "10k BOOT0 pull-down on PA14/SWCLK"
- note added: "10k pull-up + 100nF on NRST"
- note added: "CC1/CC2 -> 5.1k to GND; D+/D- via 22R series; VBUS_SENSE via 100k/100k divider."
- note added: "RN4871-I_RM128 Bluetooth Low Energy"
- note added: "R_BLE_RST 100R in series on BLE_RST line"
- note added: "SWD Debug — Samtec FTSH-107 (J3)"
- note added: "USB-C Connector (J2)"

Commit message: Schematic finalized
Parts:
- removed C10: 1uF, sldrnrd:C_0603, symbol sldrnrd:Capacitor/C_0603
- removed C11, C22: 10nF, sldrnrd:C_0603, symbol sldrnrd:Capacitor/C_0603
- removed C12, C21, C7, C8: 100nF, sldrnrd:C_0603, symbol sldrnrd:Capacitor/C_0603
- removed C19: 10uF, sldrnrd:C_0805, symbol sldrnrd:Capacitor/C_0805
- removed C9: 4.7uF, sldrnrd:C_0805, symbol sldrnrd:Capacitor/C_0805
- removed J2: USB-C, sldrnrd:USB_C, symbol sldrnrd:Connector/USB/USB_C
- removed J3: FTSH-107-01-L-DV-K, sldrnrd:HDR-SMD_14P-P1.27_FTSH-107-01-L-DV-K, symbol sldrnrd:Connector/50Mil/Header_50mil_2x07
- removed R8: 100R, sldrnrd:R_0603, symbol sldrnrd:Resistor/R_0603
- removed U11: LM35DGS, sldrnrd:SOT-23, symbol sldrnrd:Sensor/LM35
- removed U9: 24LC256-I_ST, sldrnrd:TSSOP-8, symbol sldrnrd:Memory/EEPROM/24LC256-I_ST
- added C17: 1uF, sldrnrd:C_0603, symbol sldrnrd:Capacitor/C_0603
- added C19, C20: 12.5p, sldrnrd:C_0603, symbol sldrnrd:Capacitor/C_0603
- added C23: 100n, sldrnrd:C_0603, symbol sldrnrd:Capacitor/C_0603
- added Y1: 32.768kHz, sldrnrd:CRYSTAL-3215, symbol sldrnrd:Crystal/Q13FC1350000400
- C18: value 100nF -> 100n
- C21: renamed from C14; value 33pF -> 20p
- C22: renamed from C13; value 33pF -> 20p
- U7: renamed from U2; LCSC (none) -> C633941; MPN (none) -> RN4871-I/RM128; Manufacturer (none) -> Microchip
- Y2: renamed from Y1; LCSC (none) -> C115962; MPN (none) -> X50328MSB2GI; Manufacturer (none) -> YXC
- renumbered U1 to U6
Connections:
- net ENC2_B is gone; now on net BLE_UART_MCU_TO_BLE: U6.25 (PC4)
- net ENC2_SW is gone; now on net BLE_UART_BLE_TO_MCU: U6.26 (PC5)
- net I2C2_SCL is gone; now on net BLE_P3_6: U6.30 (PB10)
- net I2C2_SDA is gone; now on net BLE_P1_7: U6.31 (PB11)
- net PCAP1_RST is gone; now on net BUZZER: U6.49 (PC9)
- net PCAP2_RST is gone; now on net DISP_CS: U6.50 (PD0)
- net BUZZER: no longer U6.57 (PB3)
- net DISP_CS: no longer U6.21 (PA4)
- net DISP_MOSI: now also U6.54 (PD4); no longer U6.24 (PA7)
- net DISP_ON: now also U6.52 (PD2); no longer U6.36 (PA8)
- net DISP_SCK: now also U6.51 (PD1); no longer U6.22 (PA5)
- net DISP_VCOM: now also U6.53 (PD3); no longer U6.23 (PA6)
- net GND: now also U6.7 (VREF+), C17.2, C19.2, C20.2, C23.2; no longer C22.1, U6.10 (PF0), U7.12 (P0_2), U7.3 (P1_2), Y2.1 (OSC1)
- net LED_PWR: now also U6.58 (PB4); no longer U6.14 (PC1)
- net TEMP_SENSE: now also U6.48 (PC8); no longer U6.28 (PB1)
- net BLE_P1_7: now reaches U7.5 (P1_7)
- net BLE_P1_6: now reaches U7.6 (P1_6)
- net BLE_P1_6: now also U6.28 (PB1)
- net BLE_P3_6: now reaches U7.9 (P3_6)
- net ENC_2B: now reaches U6.1 (PC11)
- net PCAP04_2_P2: now reaches U6.16 (PC3)
- net ENC_2A: now reaches U6.2 (PC12)
- net BLE_P0_2: now reaches U6.29 (PB2)
- net BLE_P0_2: now also U7.12 (P0_2)
- net ENC_2SW: now reaches U6.3 (PC13)
- net at U6.4 (PC14): now also C19.1, Y1.2 (OSC2)
- net DEBUG_UART_MCU_TO_PC: now reaches U6.40 (PD8)
- net DEBUG_UART_PC_TO_MCU: now reaches U6.41 (PD9)
- net STANDBY_SENSE: now reaches U6.55 (PD5)
- net CHARGE_SENSE: now reaches U6.56 (PD6)
- net LED_STATUS: now reaches U6.59 (PB5)
- net ~{ENC_1SW}: now reaches U6.64 (PC10)
- removed net +3V3: C18.1, U6.5 (PC15), U6.6 (VBAT), U6.7 (VREF+), U6.8 (VDD), U7.14 (VBAT), U7.15 (P2_7), U7.16 (P2_0)
- net BLE_RST renamed BATTERY_SENSE
- net BATTERY_SENSE: no longer U7.10 (RST_N)
- net BLE_RX renamed BLE_UART_BLE_TO_MCU
- net BLE_UART_BLE_TO_MCU: no longer U6.61 (PB7)
- net BLE_STATUS: no longer names the net of U7.11 (P0_0)
- net BLE_STATUS: no longer U6.48 (PC8)
- net BLE_TX renamed BLE_UART_MCU_TO_BLE
- net BLE_UART_MCU_TO_BLE: no longer U6.60 (PB6)
- net CHG_SENSE renamed PCAP04_1_INT
- net ENC1_A renamed PCAP04_2_INT
- net ENC1_B renamed 3V3_EN
- net ENC1_SW renamed 5V_EN
- net ENC2_A renamed ~{CHARGE_EN}
- net I2C1_SCL renamed ENC_1B
- net I2C1_SDA renamed ENC_1A
- net LDO_EN renamed PCAP04_2_SCL
- net LED_STS renamed PCAP04_2_P3
- net NRST renamed ~{RST}
- net OSC_OUT: no longer names the net of C21.1, Y2.2 (OSC2)
- net OSC_OUT: now also U6.10 (PF0); no longer U6.11 (PF1)
- net PCAP1_INT: no longer names the net of U6.38 (PC6)
- net PCAP2_INT: no longer names the net of U6.39 (PC7)
- net SCL_CS renamed BLE_P2_0
- net BLE_P2_0: now also U7.16 (P2_0)
- net SPI2_MISO renamed PCAP04_1_SDA
- net SPI2_MOSI renamed PCAP04_1_P2
- net SPI2_SCK renamed PCAP04_1_SCL
- net USB_DM renamed USB_D-
- net USB_DP renamed USB_D+
- net VBAT_SENSE renamed ~{BLE_RST}
- net ~{BLE_RST}: now also U7.10 (RST_N)
- new net: C22.1, U6.11 (PF1), Y2.1 (OSC1)
- new net: C20.1, U6.5 (PC15), Y1.1 (OSC1)
- new net EEPROM_SCL: U6.60 (PB6)
- new net EEPROM_SDA: U6.61 (PB7)
- new net PCAP04_1_P3: U6.36 (PA8)
- new net PCAP04_2_SDA: U6.14 (PC1)
- new net SCL3300_CS: U6.21 (PA4)
- new net SCL3300_MISO: U6.23 (PA6)
- new net SCL3300_MOSI: U6.24 (PA7)
- new net SCL3300_SCK: U6.22 (PA5)
- new net SWO: U6.57 (PB3)
- new net VCC: C17.1, C18.1, C23.1, U6.8 (VDD), U7.14 (VBAT)
- no-connect marks 13 -> 0
Other:
- note added: "I2C1"
- note added: "I2C2"
- note added: "I2C3"
- note added: "SPI1"
- note added: "SPI2"
- note added: "UART1"
- note added: "UART3"
- note removed: "100R series on SWDIO/SWCLK"
- note removed: "10k BOOT0 pull-down on PA14/SWCLK"
- note removed: "10k pull-up + 100nF on NRST"
- note removed: "8 MHz Crystal"
- note removed: "CC1/CC2 -> 5.1k to GND; D+/D- via 22R series; VBUS_SENSE via 100k/100k divider."
- note removed: "Decoupling capacitors"
- note removed: "R_BLE_RST 100R in series on BLE_RST line"
- note removed: "SWD Debug — Samtec FTSH-107 (J3)"
- note removed: "USB-C Connector (J2)"
- moved on the sheet: U6, U7
