File: KiCad/mcu.kicad_sch (KiCad schematic)
At the start: 11 parts, among them U6 STM32G0B1RET6, U7 RN4871-I_RM128, Y1 32.768kHz, Y2 8MHz

Commit message: Restore manual KiCad edits lost in 2026-05-10 force-push reset
Recovers connectors/mcu/power/ui schematics and the PCB layout from the
manual saves captured in KiCad/.history/ (timestamp 2026-05-10 19:55),
which were wiped when the working tree was hard-reset to origin/master
after an amended Schematic finalized force-push.

Co-Authored-By: Claude Opus 4.7 <noreply@anthropic.com>
Parts:
- added C18: 100n, sldrnrd:C_0603, symbol sldrnrd:Capacitor/C_0603
- renumbered C17 to C16, C18 to C17
Connections:
- net 3V3_EN is gone; now on net PCAP04_2_INT: U6.18 (PA1)
- net ~{ENC_1SW} is gone; now on net LED_PWR: U6.64 (PC10)
- net 5V_EN: now also U6.39 (PC7); no longer U6.19 (PA2)
- net GND: now also C18.2; no longer U6.7 (VREF+)
- net LED_PWR: no longer U6.58 (PB4)
- net LED_STATUS: now also U6.58 (PB4); no longer U6.59 (PB5)
- net PCAP04_2_INT: no longer U6.17 (PA0)
- net VBUS_SENSE: now also U6.19 (PA2); no longer U6.42 (PA10)
- net  ~{3v3_EN}: now reaches U6.38 (PC6)
- net 3V3_STANDBY: now reaches U6.6 (VBAT)
- net 3V3_STANDBY: now also C16.1, C17.1, U6.7 (VREF+), U6.8 (VDD), C18.1
- removed net VCC: C16.1, C17.1, C23.1, U6.8 (VDD), U7.14 (VBAT)
- new net 3V3: C23.1, U7.14 (VBAT)
- new net ENC_1SW: U6.59 (PB5)
Other:
- note added: "wakeup"
- note added: "wakeup 2"
- note added: "wakeup 4"
- note added: "wakeup 6"
- moved on the sheet: C16, C17
