File: KiCad/mcu.kicad_sch (KiCad schematic)
At the start: 12 parts, among them U6 STM32G0B1RET6, U7 RN4871-I_RM128, Y1 32.768kHz, Y2 8MHz

Commit message: Basic board layout changed. MCU pinout changed accordingly
Connections:
- net BLE_P0_2: now also U6.58 (PB4); no longer U6.29 (PB2)
- net BLE_P1_6: now also U6.2 (PC12); no longer U6.28 (PB1)
- net BLE_P1_7: now also U6.59 (PB5); no longer U6.31 (PB11)
- net BLE_P2_0: now also U6.3 (PC13); no longer U6.32 (PB12)
- net BLE_P3_6: now also U6.64 (PC10); no longer U6.30 (PB10)
- net BLE_UART_BLE_TO_MCU: now also U6.63 (PB9); no longer U6.26 (PC5)
- net BLE_UART_MCU_TO_BLE: now also U6.62 (PB8); no longer U6.25 (PC4)
- net ENC_1A: now also U6.25 (PC4); no longer U6.63 (PB9)
- net ENC_1B: now also U6.27 (PB0); no longer U6.62 (PB8)
- net ENC_1SW: now also U6.17 (PA0); no longer U6.59 (PB5)
- net ENC_2A: now also U6.28 (PB1); no longer U6.2 (PC12)
- net ENC_2B: now also U6.29 (PB2); no longer U6.1 (PC11)
- net ENC_2SW: now also U6.26 (PC5); no longer U6.3 (PC13)
- net LED_PWR: now also U6.32 (PB12); no longer U6.64 (PC10)
- net LED_STATUS: now also U6.31 (PB11); no longer U6.58 (PB4)
- net ~{BLE_RST}: now also U6.1 (PC11); no longer U6.27 (PB0)
Other:
- note added: "UART6"
- note added: "wakeup 1"
- note added: "wakeup 5"
- note removed: "UART1"
- note removed: "wakeup"

Commit message: Board largely routed, except power and gnd
Connections:
- net BLE_P1_6: now also U6.3 (PC13); no longer U6.2 (PC12)
- net BLE_P2_0: now also U6.1 (PC11); no longer U6.3 (PC13)
- net CHARGE_SENSE: now also U6.20 (PA3); no longer U6.56 (PD6)
- net PCAP04_1_P2: now also U6.36 (PA8); no longer U6.35 (PB15)
- net PCAP04_1_P3: now also U6.35 (PB15); no longer U6.36 (PA8)
- net ~{BLE_RST}: now also U6.2 (PC12); no longer U6.1 (PC11)
- net ~{CHARGE_EN}: now also U6.56 (PD6); no longer U6.20 (PA3)

Commit message: Environmental sensor added, mostly routed.
Parts:
- U6: LCSC (none) -> C2829307
Changed lines of the file:
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@@
 		)
 		(property "Footprint" "sldrnrd:RN4871"
-			(at 317.5 147.32 0)
+			(at 317.5 149.86 0)
 			(hide yes)
 			(show_name no)
@@
 		)
 		(property "Manufacturer" "Microchip"
-			(at 317.5 152.4 0)
+			(at 317.5 153.67 0)
 			(hide yes)
 			(show_name no)
@@
 	)
 	(symbol
-		(lib_name "Capacitor/C_0603_2")
 		(lib_id "sldrnrd:Capacitor/C_0603")
 		(at 88.9 139.7 270)
@@
 			)
 		)
-		(property "Datasheet" ""
+		(property "Datasheet" "~"
 			(at 88.9 139.7 0)
 			(hide yes)
@@
 			)
 		)
-		(property "Description" ""
+		(property "Description" "Capacitor"
 			(at 88.9 139.7 0)
 			(hide yes)
@@
 	)
 	(symbol
-		(lib_name "Capacitor/C_0603_1")
 		(lib_id "sldrnrd:Capacitor/C_0603")
 		(at 88.9 106.68 270)
@@
 			)
 		)
-		(property "Datasheet" ""
+		(property "Datasheet" "~"
 			(at 88.9 106.68 0)
 			(hide yes)
@@
 			)
 		)
-		(property "Description" ""
+		(property "Description" "Capacitor"
 			(at 88.9 106.68 0)
 			(hide yes)
@@
 		)
 		(property "Footprint" "sldrnrd:LQFP-64"
-			(at 160.02 127 0)
+			(at 165.1 127 0)
 			(hide yes)
 			(show_name no)
@@
 		)
 		(property "Datasheet" "${SLDRNRD_LIB}/datasheets/Microcontroller/STM/STM32G0B1.pdf"
-			(at 160.02 127 0)
+			(at 173.99 127 0)
 			(hide yes)
 			(show_name no)
@@
 		)
 		(property "Description" "STM32G0B1RET6 ARM Cortex-M0+ 64MHz 512KB Flash"
-			(at 160.02 127 0)
+			(at 173.99 127 0)
+			(hide yes)
+			(show_name no)
+			(do_not_autoplace no)
+			(effects
+				(font
+					(size 1.27 1.27)
+				)
+			)
+		)
+		(property "LCSC" "C2829307"
+			(at 162.56 127 0)
 			(hide yes)
 			(show_name no)
@@
 	)
 	(symbol
-		(lib_name "Capacitor/C_0603_2")
 		(lib_id "sldrnrd:Capacitor/C_0603")
 		(at 88.9 116.84 270)
@@
 			)
 		)
-		(property "Datasheet" ""
+		(property "Datasheet" "~"
 			(at 88.9 116.84 0)
 			(hide yes)
@@
 			)
 		)
-		(property "Description" ""
+		(property "Description" "Capacitor"
 			(at 88.9 116.84 0)
 			(hide yes)
@@
 	)
 	(symbol
-		(lib_name "Capacitor/C_0603_1")
 		(lib_id "sldrnrd:Capacitor/C_0603")
 		(at 71.12 133.35 0)
@@
 			)
 		)
-		(property "Datasheet" ""
+		(property "Datasheet" "~"
 			(at 71.12 133.35 0)
 			(hide yes)
@@
 			)
 		)
-		(property "Description" ""
+		(property "Description" "Capacitor"
 			(at 71.12 133.35 0)
 			(hide yes)
@@
 	)
 	(symbol
-		(lib_name "Capacitor/C_0603_1")
 		(lib_id "sldrnrd:Capacitor/C_0603")
 		(at 373.38 143.51 0)
@@
 			)
 		)
-		(property "Datasheet" ""
+		(property "Datasheet" "~"
 			(at 373.38 143.51 0)
 			(hide yes)
@@
 			)
 		)
-		(property "Description" ""
+		(property "Description" "Capacitor"
 			(at 373.38 143.51 0)
 			(hide yes)
@@
 	)
 	(symbol
-		(lib_name "Capacitor/C_0603_1")
 		(lib_id "sldrnrd:Capacitor/C_0603")
 		(at 88.9 129.54 270)
@@
 			)
 		)
-		(property "Datasheet" ""
+		(property "Datasheet" "~"
 			(at 88.9 129.54 0)
 			(hide yes)
@@
 			)
 		)
-		(property "Description" ""
+		(property "Description" "Capacitor"
 			(at 88.9 129.54 0)
 			(hide yes)
@@
 	)
 	(symbol
-		(lib_name "Capacitor/C_0603_3")
 		(lib_id "sldrnrd:Capacitor/C_0603")
 		(at 52.07 133.35 0)
@@
 			)
 		)
-		(property "Datasheet" ""
+		(property "Datasheet" "~"
 			(at 52.07 133.35 0)
 			(hide yes)
@@
 			)
 		)
-		(property "Description" ""
+		(property "Description" "Capacitor"
 			(at 52.07 133.35 0)
 			(hide yes)
@@
 	)
 	(symbol
-		(lib_name "Capacitor/C_0603_1")
 		(lib_id "sldrnrd:Capacitor/C_0603")
 		(at 62.23 133.35 0)
@@
 			)
 		)
-		(property "Datasheet" ""
+		(property "Datasheet" "~"
 			(at 62.23 133.35 0)
 			(hide yes)
@@
 			)
 		)
-		(property "Description" ""
+		(property "Description" "Capacitor"
 			(at 62.23 133.35 0)
 			(hide yes)

Commit message: External temperature sensor added
Connections:
- net TEMP_SENSE_EXT: now reaches U6.42 (PA10)
Changed lines of the file:
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@@
+	(wire
+		(pts
+			(xy 200.66 120.65) (xy 205.74 120.65)
+		)
+		(stroke
+			(width 0)
+			(type default)
+		)
+	)
 	(wire
 		(pts
@@
 			)
 		)
+	)
+	(global_label "TEMP_SENSE_EXT"
+		(shape input)
+		(at 205.74 120.65 0)
+		(effects
+			(font
+				(size 1.27 1.27)
+			)
+			(justify left)
+		)
+		(property "Intersheetrefs" "${INTERSHEET_REFS}"
+			(at 205.74 120.65 0)
+			(show_name no)
+			(do_not_autoplace no)
+			(effects
+				(font
+					(size 1.27 1.27)
+				)
+			)
+		)
+		(property "Intersheetref" "${INTERSHEET_REFS}"
+			(at 205.74 120.65 0)
+			(hide yes)
+			(show_name no)
+			(do_not_autoplace no)
+			(effects
+				(font
+					(size 1.27 1.27)
+				)
+			)
+		)

Commit message: Capacitors changed to specific symbols, board layout not yet complete
Parts:
- C16: value 1uF -> 1u; footprint sldrnrd:C_0603 -> sldrnrd:C_0805; symbol sldrnrd:Capacitor/C_0603 -> sldrnrd:Capacitor/C0805_1u; Dielectric (none) -> X7R; LCSC (none) -> C28323; MPN (none) -> CL21B105KBFNNNE; Manufacturer (none) -> Samsung; Voltage (none) -> 50V
- C17, C18, C23: symbol sldrnrd:Capacitor/C_0603 -> sldrnrd:Capacitor/C0603_100n; Dielectric (none) -> X7R; LCSC (none) -> C14663; MPN (none) -> CC0603KRX7R9BB104; Manufacturer (none) -> Yageo; Voltage (none) -> 50V
- C19, C20: value 12.5p -> 12p5; symbol sldrnrd:Capacitor/C_0603 -> sldrnrd:Capacitor/C0603_12p5; Dielectric (none) -> C0G; Voltage (none) -> 50V
- C21, C22: symbol sldrnrd:Capacitor/C_0603 -> sldrnrd:Capacitor/C0603_20p; Dielectric (none) -> C0G; LCSC (none) -> C1648; MPN (none) -> CL10C200JB8NNNC; Manufacturer (none) -> Samsung; Voltage (none) -> 50V
