File: KiCad/power.kicad_sch (KiCad schematic)
At the start: 21 parts, among them Q1 FS8205A, Q3 DMG2305UX, U10 TP4056, U3 TP4056, U4 DW01A, U5 LP5907MFX-3.3, U6 SD6210A, U7 LP5907MFX-3.3

Commit message: Schematics edited manually
Parts:
- removed C4, C7: 1uF, sldrnrd:C_0603, symbol sldrnrd:Capacitor/C_0603
- removed C8: 10uF, sldrnrd:C_0603, symbol sldrnrd:Capacitor/C_0603
- removed R4: 100k, sldrnrd:R_0603, symbol sldrnrd:Resistor/R_0603
- removed U10: TP4056, sldrnrd:ESOP-8, symbol sldrnrd:Power/BatteryManagement/TP4056
- removed U7: LP5907MFX-3.3, sldrnrd:SOT-23-5, symbol sldrnrd:Power/LinearRegulator/LP5907MFX-3.3_NOPB
- added C23, C30, C31, C32, C33, C38, C39: 100n, sldrnrd:C_0603, symbol sldrnrd:Capacitor/C_0603
- added C24: 10u, sldrnrd:C_0603, symbol sldrnrd:Capacitor/C_0603
- added C25, C26: 1uF, sldrnrd:C_0603, symbol sldrnrd:Capacitor/C_0603
- added C27, C28: 10u, sldrnrd:C_0805, symbol sldrnrd:Capacitor/C_0805
- added C29: 3u3, sldrnrd:C_0805, symbol sldrnrd:Capacitor/C_0805
- added C34, C35, C36, C37: 10n, sldrnrd:C_0603, symbol sldrnrd:Capacitor/C_0603
- added D3: LED_Red_0603, sldrnrd:LED_0603, symbol sldrnrd:LED/LED_Red_0603
- added D4: LED_Green_0603, sldrnrd:LED_0603, symbol sldrnrd:LED/LED_Green_0603
- added D5, D6, D7: BAT54WS, sldrnrd:SOD-323, symbol sldrnrd:Diode/BAT54WS
- added J1: JST_PH_2.0mm_1x02, sldrnrd:JST_PH_2.0mm_1x02, symbol sldrnrd:Connector/JST/JST_PH_2.0mm_1x02
- added Q2: AO3400A, sldrnrd:SOT-23, symbol sldrnrd:Transistor/MosfetN/AO3400A
- added R10, R12: 1k, sldrnrd:R_0603, symbol sldrnrd:Resistor/R_0603
- added R11, R15, R16, R21, R22, R23, R28, R30: 33k, sldrnrd:R_0603, symbol sldrnrd:Resistor/R_0603
- added R13: 100k, sldrnrd:R_0603, symbol sldrnrd:Resistor/R_0603
- added R14, R17, R18, R19, R20, R24, R29: 68k, sldrnrd:R_0603, symbol sldrnrd:Resistor/R_0603
- added R9: 2k, sldrnrd:R_0603, symbol sldrnrd:Resistor/R_0603
- added SW1, SW2: PEC11R-4215F-S0024, sldrnrd:RotaryEncoder_PEC11R, symbol sldrnrd:InputDevice/RotaryEncoder/PEC11R-4215F-S0024
- added U10: LP5907MFX-3.3/NOPB, sldrnrd:SOT-23-5, symbol sldrnrd:Power/LinearRegulator/LP5907MFX-3.3_NOPB
- added U8: SN74HC14PWR, sldrnrd:TSSOP-14, symbol sldrnrd:Logic/74/SN74HC14PWR
- C1: value 10uF -> 10u
- C3: value 10uF -> 1uF
- C5: value 10uF -> 100n
- C6: value 100nF -> 100n
- R2: value 2.4k -> 2k4
- R5: value 390k -> 68k
- U4: LCSC (none) -> C85680; MPN (none) -> DW01A; Manufacturer (none) -> Fortune Semicon
- U5: value LP5907MFX-3.3 -> LP5907MFX-3.3/NOPB; LCSC (none) -> C80670; MPN (none) -> LP5907MFX-3.3/NOPB; Manufacturer (none) -> TI
- U6: LCSC (none) -> C250809; MPN (none) -> SD6210A; Manufacturer (none) -> SHOUDING
Connections:
- net VBAT_RAW is gone; now on net VCC: Q3.2 (S)
- net at U4.2 (CS): now also R9.1; no longer R3.2
- net STANDBY_SENSE: now reaches U3.6 (~{STDBY})
- net STANDBY_SENSE: now also D4.2 (K)
- net +3V3 renamed GND
- net GND: now also C24.2, C25.2, C26.2, C27.2, C28.2, C30.2, C31.2, C32.2, C33.2, C34.2, C35.2, C36.2, C37.2, C38.2, C39.2, Q2.2 (S), R11.2, R29.2, R9.2, SW1.2 (COM), SW2.2 (COM), SW2.4 (SW1), U10.2 (GND), U8.7 (GND); no longer C1.1, C3.1, C6.1, R1.1, R2.2, R3.1, U3.2 (PROG), U3.4 (VCC), U3.8 (CE), U5.3 (EN), U5.5 (OUT), U6.3 (EN)
- net +5V renamed 5V0
- net 5V0: now also C27.1
- net CELL_NEG renamed BAT-
- net BAT-: now also R1.1, C23.2, J1.2
- net CFLY_N: no longer names the net of U6.4 (C-)
- net CFLY_N: now also C29.2
- net CHG_SENSE renamed CHARGE_SENSE
- net CHARGE_SENSE: now also D3.2 (K)
- net DW01_VDD: no longer names the net of U4.5 (VCC)
- net DW01_VDD: now also R3.1, C23.1
- net PROT_OC: no longer names the net of Q1.5 (G2), U4.3 (OC)
- net PROT_OD: no longer names the net of Q1.4 (G1), U4.1 (OD)
- net VBAT renamed VCC
- net VCC: now also R3.2, C24.1, C25.1, C28.1, C30.1, R13.1, SW1.4 (SW1), U10.1 (IN); no longer Q3.3 (D), U6.6 (C+)
- net VBAT_SENSE renamed BATTERY_SENSE
- net BATTERY_SENSE: now also C6.1, R13.2
- new net: R19.2, R22.2, SW2.1 (A)
- new net: R16.2, R18.2, SW1.3 (B)
- new net: D3.1 (A), R10.2
- new net: D5.1 (K), D6.1 (K), D7.1 (K), R29.1, R30.1
- new net: R23.2, R24.1, SW2.5 (SW2)
- new net: Q2.3 (D), R28.2, U3.8 (CE)
- new net: C29.1, U6.6 (C+)
- new net: D4.1 (A), R12.2
- new net: R15.2, R17.2, SW1.1 (A)
- new net: R20.2, R21.2, SW2.3 (B)
- new net: R2.2, U3.2 (PROG)
- new net 3V3: C3.1, C31.1, C39.1, R10.1, R12.1, R15.1, R16.1, R21.1, R22.1, R23.1, U5.5 (OUT), U8.14 (VCC)
- new net 3V3_EN: D7.2 (A)
- new net 3V3_Sensors: C26.1, C33.1, U10.5 (OUT)
- new net 5V_EN: U6.3 (EN)
- new net BAT+: J1.1, Q3.3 (D)
- new net ENC_1A: U8.2 (1Y)
- new net ENC_1B: U8.4 (2Y)
- new net ENC_1SW_RAW: C32.1, R14.2, U8.5 (3A)
- new net ENC_2A: U8.8 (4Y)
- new net ENC_2B: U8.10 (5Y)
- new net ENC_2SW: U8.12 (6Y)
- new net LDO_EN: R30.2, U10.3 (EN), U5.3 (EN)
- new net PWR_ON: D6.2 (A), R11.1, R14.1, SW1.5 (SW2)
- new net V_USB: C1.1, D5.2 (A), R28.1, U3.4 (VCC)
- new net ~{CHARGE_EN}: Q2.1 (G)
- new net ~{ENC_1A_RAW}: C35.1, R17.1, U8.1 (1A)
- new net ~{ENC_1B_RAW}: C34.1, R18.1, U8.3 (2A)
- new net ~{ENC_1SW}: U8.6 (3Y)
- new net ~{ENC_2A_RAW}: C36.1, R19.1, U8.9 (4A)
- new net ~{ENC_2B_RAW}: C37.1, R20.1, U8.11 (5A)
- new net ~{ENC_2SW_RAW}: C38.1, R24.2, U8.13 (6A)
- no-connect marks 4 -> 3
Other:
- note added: "Encoder 1"
- note added: "Encoder Debouncing"
- note added: "LP5907MFX-3.3 LDO for sensors"
- note added: "Power-on logic"
- note removed: "J1 Battery"
- note removed: "LP5907MFX-3.3 LDO (Sensor)"
- moved on the sheet: C1, Q1, Q3, R1, R3, U3, U4, U5

Commit message: Schematic finalized
Parts:
- removed C32, C38, C39: 100n, sldrnrd:C_0603, symbol sldrnrd:Capacitor/C_0603
- removed C34, C35, C36, C37: 10n, sldrnrd:C_0603, symbol sldrnrd:Capacitor/C_0603
- removed R11, R15, R16, R21, R22, R23: 33k, sldrnrd:R_0603, symbol sldrnrd:Resistor/R_0603
- removed R14, R17, R18, R19, R20, R24, R29: 68k, sldrnrd:R_0603, symbol sldrnrd:Resistor/R_0603
- removed SW1, SW2: PEC11R-4215F-S0024, sldrnrd:RotaryEncoder_PEC11R, symbol sldrnrd:InputDevice/RotaryEncoder/PEC11R-4215F-S0024
- removed U8: SN74HC14PWR, sldrnrd:TSSOP-14, symbol sldrnrd:Logic/74/SN74HC14PWR
- added C1: 100n, sldrnrd:C_0603, symbol sldrnrd:Capacitor/C_0603
- added D4: BAT54WS, sldrnrd:SOD-323, symbol sldrnrd:Diode/BAT54WS
- added Q4: AO3400A, sldrnrd:SOT-23, symbol sldrnrd:Transistor/MosfetN/AO3400A
- R2: renamed from R30; value 33k -> 10k
- R5: renamed from R2; value 2k4 -> 2k
- renumbered C26 to C10, C27 to C11, C5 to C12, C30 to C13, C6 to C14, C28 to C15, C29 to C16, C23 to C3, C31 to C4, C3 to C5, C1 to C6, C25 to C7, C24 to C8, C33 to C9, D5 to D1, D6 to D2, D7 to D3, D3 to D5, D4 to D6, Q3 to Q1, Q1 to Q2, Q2 to Q3, R5 to R10, R9 to R3, R3 to R4, R28 to R6, R10 to R7, R12 to R8, R13 to R9, U4 to U1, U5 to U2, U10 to U4, U6 to U5
Connections:
- net 3V3: now also Q4.1 (G)
- net GND: now also C1.2, Q4.2 (S); no longer R10.2
- net LDO_EN: now also C1.1, D4.2 (A)
- net VCC: now also D4.1 (K)
- new net: Q4.3 (D), R10.2
Other:
- note removed: "Encoder 1"
- note removed: "Encoder Debouncing"
- moved on the sheet: C14, R2
