File: KiCad/power.kicad_sch (KiCad schematic)
At the start: 42 parts, among them J1 JST_PH_2.0mm_1x02, Q1 DMG2305UX, Q2 FS8205A, Q3 AO3400A, Q4 AO3400A, U1 DW01A, U2 LP5907MFX-3.3/NOPB, U3 TP4056, U4 LP5907MFX-3.3/NOPB, U5 SD6210A

Commit message: Restore manual KiCad edits lost in 2026-05-10 force-push reset
Recovers connectors/mcu/power/ui schematics and the PCB layout from the
manual saves captured in KiCad/.history/ (timestamp 2026-05-10 19:55),
which were wiped when the working tree was hard-reset to origin/master
after an amended Schematic finalized force-push.

Co-Authored-By: Claude Opus 4.7 <noreply@anthropic.com>
Parts:
- removed C1: 100n, sldrnrd:C_0603, symbol sldrnrd:Capacitor/C_0603
- removed C10, C5: 1uF, sldrnrd:C_0603, symbol sldrnrd:Capacitor/C_0603
- removed D1, D2, D3, D4: BAT54WS, sldrnrd:SOD-323, symbol sldrnrd:Diode/BAT54WS
- removed R2: 10k, sldrnrd:R_0603, symbol sldrnrd:Resistor/R_0603
- added C4, C9: 10u, sldrnrd:C_0805, symbol sldrnrd:Capacitor/C_0805
- added Q3: DMG2305UX, sldrnrd:SOT-23-BR, symbol sldrnrd:Transistor/MosfetP/DMG2305UX-13
- renumbered C2 to C1, C11 to C10, C12 to C11, C13 to C12, C14 to C13, C15 to C14, C16 to C15, C4 to C2, C6 to C5, C7 to C6, C8 to C7, C9 to C8, D5 to D1, D6 to D2, Q3 to Q4, Q4 to Q5, R3 to R2, R4 to R3, R5 to R4, R6 to R5, R7 to R6, R8 to R7, R9 to R8, R10 to R9
Connections:
- net 3V3: now also U4.3 (EN), Q3.3 (D); no longer C2.1, U2.5 (OUT)
- net 3V3_Sensors: now also C9.1
- net GND: now also C4.2, C9.2
- net VCC: now also U2.3 (EN)
- removed net LDO_EN: U2.3 (EN), U4.3 (EN)
- new net  ~{3v3_EN}: Q3.1 (G)
- new net 3V3_STANDBY: C2.1, C4.1, Q3.2 (S), U2.5 (OUT)
Other:
- note removed: "Power-on logic"
- moved on the sheet: C1, C2, U2
