File: KiCad/power.kicad_sch (KiCad schematic)
At the start: 37 parts, among them J1 JST_PH_2.0mm_1x02, Q1 DMG2305UX, Q2 FS8205A, Q3 DMG2305UX, Q4 AO3400A, Q5 AO3400A, U1 DW01A, U2 LP5907MFX-3.3/NOPB, U3 TP4056, U4 LP5907MFX-3.3/NOPB, U5 SD6210A

Commit message: Environmental sensor added, mostly routed.
Parts:
- Q1, Q3: footprint sldrnrd:SOT-23-BR -> sldrnrd:SOT-23-3; LCSC (none) -> C144153; MPN (none) -> DMG2305UX-13; Manufacturer (none) -> Diodes Inc.
- Q2: LCSC (none) -> C14212; MPN (none) -> FS8205A; Manufacturer (none) -> Fortune Semicon
- Q4, Q5: footprint sldrnrd:SOT-23 -> sldrnrd:SOT-23-3
- R3, R6, R7: symbol sldrnrd:Resistor/R_0603 -> sldrnrd:Resistor/R0603_1k; LCSC (none) -> C21190; MPN (none) -> 0603WAF1001T5E; Manufacturer (none) -> Uni-Royal
Connections:
- net 3V3: now also D1.1 (A), D2.1 (A); no longer R6.1, R7.1
- net CHARGE_SENSE: now also R6.2; no longer D1.2 (K)
- net STANDBY_SENSE: now also R7.2; no longer D2.2 (K)
- new net: D1.2 (K), R6.1
- new net: D2.2 (K), R7.1
Other:
- moved on the sheet: D1, D2, R6, R7

Commit message: JST headers fixed, no more errors, fully routed
Parts:
- R1, R8: symbol sldrnrd:Resistor/R_0603 -> sldrnrd:Resistor/R0603_100k; LCSC (none) -> C25803; MPN (none) -> 0603WAF1003T5E; Manufacturer (none) -> Uni-Royal
Changed lines of the file:
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@@
 	)
 	(symbol
-		(lib_id "sldrnrd:Resistor/R_0603")
+		(lib_id "sldrnrd:Resistor/R0603_100k")
 		(at 483.87 60.96 0)
 		(unit 1)
@@
 		(dnp no)
 		(property "Reference" "R8"
-			(at 481.584 62.23 90)
-			(show_name no)
-			(do_not_autoplace no)
-			(effects
-				(font
-					(size 1.27 1.27)
-				)
-				(justify left)
+			(at 485.902 60.96 90)
+			(show_name no)
+			(do_not_autoplace no)
+			(effects
+				(font
+					(size 1.27 1.27)
+				)
 			)
 		)
 		(property "Value" "100k"
-			(at 486.41 63.5 90)
-			(show_name no)
-			(do_not_autoplace no)
-			(effects
-				(font
-					(size 1.27 1.27)
-				)
-				(justify left)
+			(at 481.838 60.96 90)
+			(show_name no)
+			(do_not_autoplace no)
+			(effects
+				(font
+					(size 1.27 1.27)
+				)
 			)
 		)
@@
 			)
 		)
-		(property "Description" "Resistor"
+		(property "Description" "100k Resistor, 0603, 1%, 75V, 100mW"
+			(at 483.87 60.96 0)
+			(hide yes)
+			(show_name no)
+			(do_not_autoplace no)
+			(effects
+				(font
+					(size 1.27 1.27)
+				)
+			)
+		)
+		(property "Manufacturer" "Uni-Royal"
+			(at 483.87 60.96 0)
+			(hide yes)
+			(show_name no)
+			(do_not_autoplace no)
+			(effects
+				(font
+					(size 1.27 1.27)
+				)
+			)
+		)
+		(property "MPN" "0603WAF1003T5E"
+			(at 483.87 60.96 0)
+			(hide yes)
+			(show_name no)
+			(do_not_autoplace no)
+			(effects
+				(font
+					(size 1.27 1.27)
+				)
+			)
+		)
+		(property "LCSC" "C25803"
 			(at 483.87 60.96 0)
 			(hide yes)
@@
 	)
 	(symbol
-		(lib_id "sldrnrd:Resistor/R_0603")
+		(lib_id "sldrnrd:Resistor/R0603_100k")
 		(at 78.74 92.71 180)
 		(unit 1)
@@
 		(dnp no)
 		(property "Reference" "R1"
-			(at 76.708 92.71 0)
-			(show_name no)
-			(do_not_autoplace no)
-			(effects
-				(font
-					(size 1.27 1.27)
-				)
-				(justify left)
+			(at 76.708 92.71 90)
+			(show_name no)
+			(do_not_autoplace no)
+			(effects
+				(font
+					(size 1.27 1.27)
+				)
 			)
 		)
 		(property "Value" "100k"
-			(at 85.344 92.71 0)
-			(show_name no)
-			(do_not_autoplace no)
-			(effects
-				(font
-					(size 1.27 1.27)
-				)
-				(justify left)
+			(at 80.772 92.71 90)
+			(show_name no)
+			(do_not_autoplace no)
+			(effects
+				(font
+					(size 1.27 1.27)
+				)
 			)
 		)
@@
 			)
 		)
-		(property "Description" "Resistor"
-			(at 78.74 92.71 0)
-			(hide yes)
+		(property "Description" "100k Resistor, 0603, 1%, 75V, 100mW"
+			(at 78.74 92.71 0)
+			(hide yes)
+			(show_name no)
+			(do_not_autoplace no)
+			(effects
+				(font
+					(size 1.27 1.27)
+				)
+			)
+		)
+		(property "Manufacturer" "Uni-Royal"
+			(at 78.74 92.71 0)
+			(hide yes)
+			(show_name no)
+			(do_not_autoplace no)
+			(effects
+				(font
+					(size 1.27 1.27)
+				)
+			)
+		)
+		(property "MPN" "0603WAF1003T5E"
+			(at 78.74 92.71 0)
+			(hide yes)
+			(show_name no)
+			(do_not_autoplace no)
+			(effects
+				(font
+					(size 1.27 1.27)
+				)
+			)
+		)
+		(property "LCSC" "C25803"
+			(at 78.74 92.71 0)
+			(hide yes)

Commit message: Capacitors changed to specific symbols, board layout not yet complete
Parts:
- C1, C6: value 1uF -> 1u; footprint sldrnrd:C_0603 -> sldrnrd:C_0805; symbol sldrnrd:Capacitor/C_0603 -> sldrnrd:Capacitor/C0805_1u; Dielectric (none) -> X7R; LCSC (none) -> C28323; MPN (none) -> CL21B105KBFNNNE; Manufacturer (none) -> Samsung; Voltage (none) -> 50V
- C10, C14, C4, C9: footprint sldrnrd:C_0805 -> sldrnrd:C_1206; symbol sldrnrd:Capacitor/C_0805 -> sldrnrd:Capacitor/C1206_10u; Dielectric (none) -> X7R; LCSC (none) -> C70462; MPN (none) -> CC1206KKX7R8BB106; Manufacturer (none) -> Yageo; Voltage (none) -> 25V
- C11, C12, C13, C2, C3, C8: symbol sldrnrd:Capacitor/C_0603 -> sldrnrd:Capacitor/C0603_100n; Dielectric (none) -> X7R; LCSC (none) -> C14663; MPN (none) -> CC0603KRX7R9BB104; Manufacturer (none) -> Yageo; Voltage (none) -> 50V
- C15: value 3u3 -> 2u2; symbol sldrnrd:Capacitor/C_0805 -> sldrnrd:Capacitor/C0805_2u2; Dielectric (none) -> X7R; LCSC (none) -> C126589; MPN (none) -> GCM21BR71C225KA64L; Manufacturer (none) -> Murata; Voltage (none) -> 16V
- C5, C7: footprint sldrnrd:C_0603 -> sldrnrd:C_1206; symbol sldrnrd:Capacitor/C_0603 -> sldrnrd:Capacitor/C1206_10u; Dielectric (none) -> X7R; LCSC (none) -> C70462; MPN (none) -> CC1206KKX7R8BB106; Manufacturer (none) -> Yageo; Voltage (none) -> 25V

Commit message: Symbols and board updated to match library
Parts:
- Q1, Q3: value DMG2305UX -> DMG2305UX-13
- R2, R4: value 2k -> R_0603
- R5: value 33k -> R_0603
- R9: value 68k -> R_0603

Commit message: Remaining resistors and capacitors replaced by specific value components
Parts:
- R2: value R_0603 -> 2k; symbol sldrnrd:Resistor/R_0603 -> sldrnrd:Resistor/R0603_2k; LCSC (none) -> C22975; MPN (none) -> 0603WAF2001T5E; Manufacturer (none) -> Uni-Royal
- R5, R9: value R_0603 -> 33k; symbol sldrnrd:Resistor/R_0603 -> sldrnrd:Resistor/R0603_33k; LCSC (none) -> C4216; MPN (none) -> 0603WAF3302T5E; Manufacturer (none) -> Uni-Royal
Changed lines of the file:
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@@
 	)
 	(symbol
-		(lib_id "sldrnrd:Resistor/R_0603")
+		(lib_id "sldrnrd:Resistor/R0603_33k")
 		(at 386.08 58.42 0)
 		(unit 1)
@@
 		(dnp no)
 		(property "Reference" "R5"
-			(at 383.794 60.452 90)
-			(show_name no)
-			(do_not_autoplace no)
-			(effects
-				(font
-					(size 1.27 1.27)
-				)
-			)
-		)
-		(property "Value" "R_0603"
-			(at 388.62 60.96 90)
+			(at 388.112 58.42 90)
+			(show_name no)
+			(do_not_autoplace no)
+			(effects
+				(font
+					(size 1.27 1.27)
+				)
+			)
+		)
+		(property "Value" "33k"
+			(at 384.048 58.42 90)
 			(show_name no)
 			(do_not_autoplace no)
@@
 			)
 		)
-		(property "Description" "Resistor"
+		(property "Description" "33k Resistor, 0603, 1%, 75V, 100mW"
+			(at 386.08 58.42 0)
+			(hide yes)
+			(show_name no)
+			(do_not_autoplace no)
+			(effects
+				(font
+					(size 1.27 1.27)
+				)
+			)
+		)
+		(property "Manufacturer" "Uni-Royal"
+			(at 386.08 58.42 0)
+			(hide yes)
+			(show_name no)
+			(do_not_autoplace no)
+			(effects
+				(font
+					(size 1.27 1.27)
+				)
+			)
+		)
+		(property "MPN" "0603WAF3302T5E"
+			(at 386.08 58.42 0)
+			(hide yes)
+			(show_name no)
+			(do_not_autoplace no)
+			(effects
+				(font
+					(size 1.27 1.27)
+				)
+			)
+		)
+		(property "LCSC" "C4216"
 			(at 386.08 58.42 0)
 			(hide yes)
@@
 	)
 	(symbol
-		(lib_id "sldrnrd:Resistor/R_0603")
+		(lib_id "sldrnrd:Resistor/R0603_2k")
 		(at 186.69 81.28 0)
 		(unit 1)
@@
 			)
 		)
-		(property "Value" "R_0603"
+		(property "Value" "2k"
 			(at 189.23 82.5499 90)
 			(show_name no)
@@
 			)
 		)
-		(property "Description" "Resistor"
+		(property "Description" "2k Resistor, 0603, 1%, 75V, 100mW"
+			(at 186.69 81.28 0)
+			(hide yes)
+			(show_name no)
+			(do_not_autoplace no)
+			(effects
+				(font
+					(size 1.27 1.27)
+				)
+			)
+		)
+		(property "Manufacturer" "Uni-Royal"
+			(at 186.69 81.28 0)
+			(hide yes)
+			(show_name no)
+			(do_not_autoplace no)
+			(effects
+				(font
+					(size 1.27 1.27)
+				)
+			)
+		)
+		(property "MPN" "0603WAF2001T5E"
+			(at 186.69 81.28 0)
+			(hide yes)
+			(show_name no)
+			(do_not_autoplace no)
+			(effects
+				(font
+					(size 1.27 1.27)
+				)
+			)
+		)
+		(property "LCSC" "C22975"
 			(at 186.69 81.28 0)
 			(hide yes)
@@
 	)
 	(symbol
-		(lib_id "sldrnrd:Resistor/R_0603")
+		(lib_id "sldrnrd:Resistor/R0603_33k")
 		(at 483.87 76.2 0)
 		(unit 1)
@@
 		(dnp no)
 		(property "Reference" "R9"
-			(at 481.584 77.47 90)
-			(show_name no)
-			(do_not_autoplace no)
-			(effects
-				(font
-					(size 1.27 1.27)
-				)
-			)
-		)
-		(property "Value" "R_0603"
-			(at 486.41 78.74 90)
+			(at 485.902 76.2 90)
+			(show_name no)
+			(do_not_autoplace no)
+			(effects
+				(font
+					(size 1.27 1.27)
+				)
+			)
+		)
+		(property "Value" "33k"
+			(at 481.838 76.2 90)
 			(show_name no)
 			(do_not_autoplace no)
@@
 			)
 		)
-		(property "Description" "Resistor"
+		(property "Description" "33k Resistor, 0603, 1%, 75V, 100mW"
 			(at 483.87 76.2 0)
 			(hide yes)
+			(show_name no)
+			(do_not_autoplace no)
+			(effects
+				(font
+					(size 1.27 1.27)
+				)
+			)
+		)
+		(property "Manufacturer" "Uni-Royal"
+			(at 483.87 76.2 0)
+			(hide yes)
+			(show_name no)
+			(do_not_autoplace no)
+			(effects
+				(font
+					(size 1.27 1.27)
+				)
+			)
+		)
+		(property "MPN" "0603WAF3302T5E"
+			(at 483.87 76.2 0)
+			(hide yes)
+			(show_name no)
+			(do_not_autoplace no)
+			(effects
+				(font
+					(size 1.27 1.27)
+				)
+			)
+		)
+		(property "LCSC" "C4216"
+			(at 483.87 76.2 0)
+			(hide yes)
