File: KiCad/ui.kicad_sch (KiCad schematic)
At the start: 12 parts, among them U12 LM35, U7 SN74AHCT244DBR

Commit message: Schematic finalized
Parts:
- removed D1: Green, sldrnrd:LED_0603, symbol sldrnrd:LED/LED_0603
- removed D2: Blue, sldrnrd:LED_0603, symbol sldrnrd:LED/LED_0603
- removed R6, R7: 330R, sldrnrd:R_0603, symbol sldrnrd:Resistor/R_0603
- removed U12: LM35, sldrnrd:SOT-23, symbol sldrnrd:Sensor/LM35
- added C24, C25, C31, C33: 10n, sldrnrd:C_0603, symbol sldrnrd:Capacitor/C_0603
- added C26, C28, C34, C35, C36: 100n, sldrnrd:C_0603, symbol sldrnrd:Capacitor/C_0603
- added D7, D8: LED_Green_0603, sldrnrd:LED_0603, symbol sldrnrd:LED/LED_Green_0603
- added R11, R12, R25: 1k, sldrnrd:R_0603, symbol sldrnrd:Resistor/R_0603
- added R13, R14, R18, R19, R20, R24: 68k, sldrnrd:R_0603, symbol sldrnrd:Resistor/R_0603
- added R15, R16, R17, R21, R22, R23: 33k, sldrnrd:R_0603, symbol sldrnrd:Resistor/R_0603
- added SW1, SW2: PEC11R-4215F-S0024, sldrnrd:RotaryEncoder_PEC11R, symbol sldrnrd:InputDevice/RotaryEncoder/PEC11R-4215F-S0024
- added U10: SN74HC14PWR, sldrnrd:TSSOP-14, symbol sldrnrd:Logic/74/SN74HC14PWR
- added U11: LM35DGS, sldrnrd:SOT-23, symbol sldrnrd:Sensor/LM35
- added U9: 24LC256-I_ST, sldrnrd:TSSOP-8, symbol sldrnrd:Memory/EEPROM/24LC256-I_ST
- renumbered C15 to C27, C40 to C29, C20 to C30, C17 to C32, U7 to U8
Connections:
- net 5V0: now also DS1.8 (EXTMODE), C35.1, U11.1 (VS+)
- net BUZZER: now also U8.11 (2A1), U8.13 (2A2), U8.15 (2A3); no longer BZ1.1
- net GND: now also C24.2, C25.2, C26.2, C28.2, C31.2, C33.2, C34.2, C35.2, C36.2, D7.2 (K), D8.2 (K), R17.2, SW1.2 (COM), SW2.2 (COM), SW2.4 (SW1), U10.7 (GND), U11.3 (GND), U9.1 (A0), U9.2 (A1), U9.3 (A2), U9.4 (VSS), U9.7 (WP); no longer DS1.8 (EXTMODE)
- net LED_PWR: now also R11.1
- net BUZZER_5V: now reaches U8.5 (2Y3)
- net BUZZER_5V: now also BZ1.1, U8.7 (2Y2), U8.9 (2Y1)
- new net: R20.2, R21.2, SW2.3 (B)
- new net: R25.2, U11.2 (VOUT)
- new net: R13.2, R16.2, SW1.1 (A)
- new net: R14.2, R15.2, SW1.3 (B)
- new net: R19.2, R22.2, SW2.1 (A)
- new net: D7.1 (A), R11.2
- new net: R23.2, R24.1, SW2.5 (SW2)
- new net: D8.1 (A), R12.2
- new net 3V3: C26.1, C36.1, R15.1, R16.1, R21.1, R22.1, R23.1, U10.14 (VCC), U9.8 (VCC)
- new net EEPROM_SCL: U9.6 (SCL)
- new net EEPROM_SDA: U9.5 (SDA)
- new net ENC_1A: U10.2 (1Y)
- new net ENC_1B: U10.4 (2Y)
- new net ENC_1SW_RAW: C28.1, R18.2, U10.5 (3A)
- new net ENC_2A: U10.8 (4Y)
- new net ENC_2B: U10.10 (5Y)
- new net ENC_2SW: U10.12 (6Y)
- new net LED_STATUS: R12.1
- new net PWR_ON: R17.1, R18.1, SW1.5 (SW2)
- new net TEMP_SENSE: R25.1
- new net VCC: SW1.4 (SW1)
- new net ~{ENC_1A_RAW}: C24.1, R13.1, U10.1 (1A)
- new net ~{ENC_1B_RAW}: C25.1, R14.1, U10.3 (2A)
- new net ~{ENC_1SW}: U10.6 (3Y)
- new net ~{ENC_2A_RAW}: C31.1, R19.1, U10.9 (4A)
- new net ~{ENC_2B_RAW}: C33.1, R20.1, U10.11 (5A)
- new net ~{ENC_2SW_RAW}: C34.1, R24.2, U10.13 (6A)
Other:
- note added: "Encoder 1"
- note added: "Encoder 2"
- note added: "Encoder Debouncing"
- note removed: "LED1 Green (Power)"
- note removed: "LED2 Blue (Status)"
- note removed: "PWM 4kHz from TIM1_CH2 (PB3)"
- moved on the sheet: BZ1, C27, C29, C30, C32, DS1, U8
