File: KiCad/ui.kicad_sch (KiCad schematic)
At the start: 38 parts, among them SW1 PEC11R-4215F-S0024, SW2 PEC11R-4215F-S0024, U10 SN74HC14PWR, U11 LM35DGS, U8 SN74AHCT244DBR, U9 24LC256-I_ST

Commit message: Restore manual KiCad edits lost in 2026-05-10 force-push reset
Recovers connectors/mcu/power/ui schematics and the PCB layout from the
manual saves captured in KiCad/.history/ (timestamp 2026-05-10 19:55),
which were wiped when the working tree was hard-reset to origin/master
after an amended Schematic finalized force-push.

Co-Authored-By: Claude Opus 4.7 <noreply@anthropic.com>
Parts:
- added R18, R19: 5k1, sldrnrd:R_0603, symbol sldrnrd:Resistor/R_0603
- DS1: footprint sldrnrd:FPC-10-1.5 -> sldrnrd:Header_FFC_1.5mm_10
- renumbered D7 to D3, D8 to D4, R11 to R10, R12 to R11, R13 to R12, R14 to R13, R15 to R14, R16 to R15, R17 to R16, R18 to R17, R19 to R20, R20 to R21, R21 to R22, R22 to R23, R23 to R24, R24 to R25, R25 to R26
Connections:
- net 3V3: now also R18.1, R19.1; no longer C36.1, R24.1, U10.14 (VCC)
- net EEPROM_SCL: now also R19.2
- net EEPROM_SDA: now also R18.2
- net GND: now also SW1.5 (SW2), SW2.5 (SW2); no longer R16.2, SW2.4 (SW1)
- net at R24.2, R25.1: now also SW2.4 (SW1); no longer SW2.5 (SW2)
- net ENC_1SW_RAW renamed ~{ENC_1SW_RAW}
- removed net PWR_ON: R16.1, R17.1, SW1.5 (SW2)
- net VCC: no longer names the net of SW1.4 (SW1)
- net VCC: now also R16.2, R17.1
- net ~{ENC_1SW} renamed ENC_1SW
- new net 3V3_STANDBY: C36.1, R16.1, R24.1, U10.14 (VCC)
Other:
- moved on the sheet: C26, C28, R16, R17, R24, R25, U9
