File: KiCad/connectors.kicad_sch (KiCad schematic)
At the start: 13 parts, among them J2 USB-C, J3 Header_FFC_1.0mm_06, J4 Header_50mil_2x07, J5 Header_FFC_1.0mm_10, J6 Header_FFC_1.0mm_10

Commit message: Restore manual KiCad edits lost in 2026-05-10 force-push reset
Recovers connectors/mcu/power/ui schematics and the PCB layout from the
manual saves captured in KiCad/.history/ (timestamp 2026-05-10 19:55),
which were wiped when the working tree was hard-reset to origin/master
after an amended Schematic finalized force-push.

Co-Authored-By: Claude Opus 4.7 <noreply@anthropic.com>
Parts:
- added C38, C40: 100n, sldrnrd:C_0603, symbol sldrnrd:Capacitor/C_0603
- added R32, R33, R35, R36: 5k1, sldrnrd:R_0603, symbol sldrnrd:Resistor/R_0603
- J2: LCSC (none) -> C165948; MPN (none) -> TYPE-C-31-M-12; Manufacturer (none) -> Korean Hroparts Elec
- renumbered C38 to C39, R26 to R27, R27 to R28, R28 to R29, R29 to R30, R30 to R31, R31 to R34
Connections:
- net 3V3: no longer J5.4, J5.6, J6.4, J6.6
- net GND: now also C38.2, C40.2
- net PCAP04_1_SCL: now also R32.2
- net PCAP04_1_SDA: now also R33.2
- net PCAP04_2_SCL: now also R35.2
- net PCAP04_2_SDA: now also R36.2
- new net 3V3_Sensors: C38.1, C40.1, J5.4, J5.6, J6.4, J6.6, R32.1, R33.1, R35.1, R36.1
Other:
- moved on the sheet: J5, J6
