File: KiCad/connectors.kicad_sch (KiCad schematic)
At the start: 19 parts, among them J2 USB-C, J3 Header_FFC_1.0mm_06, J4 Header_50mil_2x07, J5 Header_FFC_1.0mm_10, J6 Header_FFC_1.0mm_10

Commit message: Encoder fixed, main parts and dimensions locked
Parts:
- added H1, H2, H3, H4: MountingHole_Pad, sldrnrd:MountingHole_3.2mm, symbol sldrnrd:MountingHole_Pad
Connections:
- net GND: now also H1.1, H2.1, H3.1, H4.1

Commit message: Board largely routed, except power and gnd
Parts:
- added C41: 100n, sldrnrd:C_0603, symbol sldrnrd:Capacitor/C_0603
Connections:
- net 3V3: now also C41.1
- net GND: now also C41.2
Changed lines of the file:
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@@
 	)
 	(junction
+		(at 69.85 189.23)
+		(diameter 0)
+		(color 0 0 0 0)
+	)
+	(junction
 		(at 204.47 199.39)
 		(diameter 0)
@@
 	(wire
 		(pts
+			(xy 69.85 189.23) (xy 77.47 189.23)
+		)
+		(stroke
+			(width 0)
+			(type default)
+		)
+	)
+	(wire
+		(pts
 			(xy 119.38 77.47) (xy 119.38 82.55)
 		)
@@
 	(wire
 		(pts
-			(xy 66.04 193.04) (xy 77.47 193.04)
+			(xy 285.75 55.88) (xy 285.75 57.15)
 		)
 		(stroke
@@
 	(wire
 		(pts
-			(xy 285.75 55.88) (xy 285.75 57.15)
+			(xy 320.04 207.01) (xy 320.04 226.06)
 		)
 		(stroke
@@
 	(wire
 		(pts
-			(xy 320.04 207.01) (xy 320.04 226.06)
+			(xy 175.26 214.63) (xy 213.36 214.63)
 		)
 		(stroke
@@
 	(wire
 		(pts
-			(xy 175.26 214.63) (xy 213.36 214.63)
+			(xy 173.99 54.61) (xy 173.99 43.18)
 		)
 		(stroke
@@
 	(wire
 		(pts
-			(xy 173.99 54.61) (xy 173.99 43.18)
+			(xy 290.83 184.15) (xy 290.83 187.96)
 		)
 		(stroke
@@
 	(wire
 		(pts
-			(xy 290.83 184.15) (xy 290.83 187.96)
+			(xy 173.99 59.69) (xy 173.99 64.77)
 		)
 		(stroke
@@
 	(wire
 		(pts
-			(xy 173.99 59.69) (xy 173.99 64.77)
+			(xy 285.75 57.15) (xy 278.13 57.15)
 		)
 		(stroke
@@
 	(wire
 		(pts
-			(xy 285.75 57.15) (xy 278.13 57.15)
+			(xy 69.85 189.23) (xy 69.85 208.28)
 		)
 		(stroke
@@
 	(wire
 		(pts
-			(xy 175.26 195.58) (xy 193.04 195.58)
+			(xy 60.96 193.04) (xy 77.47 193.04)
 		)
 		(stroke
@@
 	(wire
 		(pts
-			(xy 180.34 181.61) (xy 180.34 187.96)
+			(xy 175.26 195.58) (xy 193.04 195.58)
 		)
 		(stroke
@@
 	(wire
 		(pts
-			(xy 278.13 77.47) (xy 278.13 82.55)
+			(xy 180.34 181.61) (xy 180.34 187.96)
 		)
 		(stroke
@@
 	(wire
 		(pts
-			(xy 198.12 67.31) (xy 198.12 78.74)
+			(xy 278.13 77.47) (xy 278.13 82.55)
 		)
 		(stroke
@@
 	(wire
 		(pts
-			(xy 82.55 76.2) (xy 82.55 82.55)
+			(xy 198.12 67.31) (xy 198.12 78.74)
 		)
 		(stroke
@@
 	(wire
 		(pts
-			(xy 52.07 64.77) (xy 50.8 64.77)
+			(xy 82.55 76.2) (xy 82.55 82.55)
 		)
 		(stroke
@@
 	(wire
 		(pts
-			(xy 66.04 200.66) (xy 77.47 200.66)
+			(xy 52.07 64.77) (xy 50.8 64.77)
 		)
 		(stroke
@@
 	(wire
 		(pts
-			(xy 66.04 204.47) (xy 77.47 204.47)
+			(xy 60.96 196.85) (xy 77.47 196.85)
 		)
 		(stroke
@@
 	(wire
 		(pts
+			(xy 69.85 213.36) (xy 69.85 215.9)
+		)
+		(stroke
+			(width 0)
+			(type default)
+		)
+	)
+	(wire
+		(pts
 			(xy 173.99 67.31) (xy 173.99 78.74)
 		)
@@
 	(wire
 		(pts
+			(xy 60.96 200.66) (xy 77.47 200.66)
+		)
+		(stroke
+			(width 0)
+			(type default)
+		)
+	)
+	(wire
+		(pts
 			(xy 330.2 191.77) (xy 330.2 233.68)
 		)
@@
 	(wire
 		(pts
-			(xy 77.47 189.23) (xy 74.93 189.23)
-		)
-		(stroke
-			(width 0)
-			(type default)
-		)
-	)
-	(wire
-		(pts
 			(xy 303.53 195.58) (xy 332.74 195.58)
 		)
@@
 	(wire
 		(pts
-			(xy 74.93 189.23) (xy 74.93 180.34)
+			(xy 69.85 189.23) (xy 69.85 180.34)
 		)
 		(stroke
@@
 	(wire
 		(pts
+			(xy 60.96 204.47) (xy 77.47 204.47)
+		)
+		(stroke
+			(width 0)
+			(type default)
+		)
+	)
+	(wire
+		(pts
 			(xy 198.12 52.07) (xy 194.31 52.07)
 		)
@@
 	(wire
 		(pts
-			(xy 66.04 196.85) (xy 77.47 196.85)
-		)
-		(stroke
-			(width 0)
-			(type default)
-		)
-	)
-	(wire
-		(pts
 			(xy 320.04 199.39) (xy 320.04 207.01)
 		)
@@
 	(global_label "SCL3300_MOSI"
 		(shape input)
-		(at 66.04 204.47 180)
+		(at 60.96 204.47 180)
 		(fields_autoplaced yes)
 		(effects
@@
 		)
 		(property "Intersheetrefs" "${INTERSHEET_REFS}"
-			(at 49.1454 204.47 0)
+			(at 44.0654 204.47 0)
 			(show_name no)
 			(do_not_autoplace no)
@@
 	(global_label "SCL3300_CS"
 		(shape input)
-		(at 66.04 193.04 180)
+		(at 60.96 193.04 180)
 		(fields_autoplaced yes)
 		(effects
@@
 		)
 		(property "Intersheetrefs" "${INTERSHEET_REFS}"
-			(at 51.2621 193.04 0)
+			(at 46.1821 193.04 0)
 			(show_name no)
 			(do_not_autoplace no)
@@
 	(global_label "SCL3300_SCK"
 		(shape input)
-		(at 66.04 196.85 180)
+		(at 60.96 196.85 180)
 		(fields_autoplaced yes)
 		(effects
@@
 		)
 		(property "Intersheetrefs" "${INTERSHEET_REFS}"
-			(at 49.9921 196.85 0)
+			(at 44.9121 196.85 0)
 			(show_name no)
 			(do_not_autoplace no)
@@
 	(global_label "SCL3300_MISO"
 		(shape output)
-		(at 66.04 200.66 180)
+		(at 60.96 200.66 180)
 		(fields_autoplaced yes)
 		(effects
@@
 		)
 		(property "Intersheetrefs" "${INTERSHEET_REFS}"
-			(at 49.1454 200.66 0)
+			(at 44.0654 200.66 0)
 			(show_name no)
 			(do_not_autoplace no)
@@
 	)
 	(symbol
+		(lib_id "sldrnrd:Power/PWR/GND")
+		(at 69.85 215.9 0)
+		(unit 1)
+		(body_style 1)
+		(exclude_from_sim no)
+		(in_bom yes)
+		(on_board yes)
+		(in_pos_files yes)
+		(dnp no)
+		(property "Reference" "#PWR0118"
+			(at 69.85 222.25 0)
+			(hide yes)
+			(show_name no)
+			(do_not_autoplace no)
+			(effects
+				(font
+					(size 1.27 1.27)
+				)
+			)
+		)
+		(property "Value" "GND"
+			(at 69.85 220.218 0)
+			(show_name no)
+			(do_not_autoplace no)
+			(effects
+				(font
+					(size 1.27 1.27)
+				)
+			)
+		)
+		(property "Footprint" ""
+			(at 69.85 215.9 0)
+			(hide yes)
+			(show_name no)
+			(do_not_autoplace no)
+			(effects
+				(font
+					(size 1.27 1.27)
+				)
+			)
+		)
+		(property "Datasheet" ""
+			(at 69.85 215.9 0)
+			(hide yes)
+			(show_name no)
+			(do_not_autoplace no)
+			(effects
+				(font
+					(size 1.27 1.27)
+				)
+			)
+		)
+		(property "Description" "Power symbol creates a global label with name \"GND\", ground"
+			(at 69.85 215.9 0)
+			(hide yes)
+			(show_name no)
+			(do_not_autoplace no)
+			(effects
+				(font
+					(size 1.27 1.27)
+				)
+			)
+		)
+		(pin "1"
+		)
+		(instances
+			(project "InclinationMeter"
+				(path "/7d35597c-fbf9-4ce7-8410-0e7922679ea3/7286337d-4cd5-4f95-b550-04c2e962fc51"
+					(reference "#PWR0118")
+					(unit 1)
+				)
+			)
+		)
+	)
+	(symbol
 		(lib_id "sldrnrd:Connector/USB/USB_C")
 		(at 64.77 60.96 0)
@@
 	)
 	(symbol
+		(lib_name "Capacitor/C_0603_2")
+		(lib_id "sldrnrd:Capacitor/C_0603")
+		(at 69.85 210.82 0)
+		(unit 1)
+		(body_style 1)
+		(exclude_from_sim no)
+		(in_bom yes)
+		(on_board yes)
+		(in_pos_files yes)
+		(dnp no)
+		(property "Reference" "C41"
+			(at 67.31 212.09 90)
+			(show_name no)
+			(do_not_autoplace no)
+			(effects
+				(font
+					(size 1.27 1.27)
+				)
+				(justify left)
+			)
+		)
+		(property "Value" "100n"
+			(at 72.898 213.106 90)
+			(show_name no)
+			(do_not_autoplace no)
+			(effects
+				(font
+					(size 1.27 1.27)
+				)
+				(justify left)
+			)
+		)
+		(property "Footprint" "sldrnrd:C_0603"
+			(at 69.85 210.82 0)
+			(hide yes)
+			(show_name no)
+			(do_not_autoplace no)
+			(effects
+				(font
+					(size 1.27 1.27)
+				)
+			)
+		)
+		(property "Datasheet" ""
+			(at 69.85 210.82 0)
+			(hide yes)
+			(show_name no)
+			(do_not_autoplace no)
+			(effects
+				(font
+					(size 1.27 1.27)
+				)
+			)
+		)
+		(property "Description" ""
+			(at 69.85 210.82 0)
+			(hide yes)
+			(show_name no)
+			(do_not_autoplace no)
+			(effects
+				(font
+					(size 1.27 1.27)
+				)
+			)
+		)
+		(pin "1"
+		)
+		(pin "2"
+		)
+		(instances
+			(project "InclinationMeter"
+				(path "/7d35597c-fbf9-4ce7-8410-0e7922679ea3/7286337d-4cd5-4f95-b550-04c2e962fc51"
+					(reference "C41")
+					(unit 1)
+				)
+			)
+		)
+	)
+	(symbol
 		(lib_id "sldrnrd:Power/PWR/GND")
 		(at 48.26 81.28 0)
@@
 	(symbol
 		(lib_id "sldrnrd:Power/PWR/3V3")
-		(at 74.93 180.34 0)
+		(at 69.85 180.34 0)
 		(unit 1)
 		(body_style 1)
@@
 		(dnp no)
 		(property "Reference" "#PWR094"
-			(at 74.93 184.15 0)
+			(at 69.85 184.15 0)
 			(hide yes)
 			(show_name no)
@@
 		)
 		(property "Value" "3V3"
-			(at 74.93 176.022 0)
+			(at 69.85 176.022 0)
 			(show_name no)
 			(do_not_autoplace no)
@@
 		)
 		(property "Footprint" ""
-			(at 74.93 180.34 0)
+			(at 69.85 180.34 0)
 			(hide yes)
 			(show_name no)
@@
 		)
 		(property "Datasheet" ""
-			(at 74.93 180.34 0)
+			(at 69.85 180.34 0)
 			(hide yes)
 			(show_name no)
@@
 		)
 		(property "Description" "Power symbol creates a global label with name \"3V3\", 3.3V supply"
-			(at 74.93 180.34 0)
+			(at 69.85 180.34 0)
 			(hide yes)
 			(show_name no)

Commit message: External temperature sensor added
Parts:
- added C43: 100n, sldrnrd:C_0603, symbol sldrnrd:Capacitor/C_0603
- added J7: Header_100mil_1x03, sldrnrd:Header_100mil_1x03, symbol sldrnrd:Connector/100Mil/Header_100mil_1x03
- added R37: 2k, sldrnrd:R_0603, symbol sldrnrd:Resistor/R_0603
Connections:
- net GND: now also C43.2, J7.2
- new net: J7.3, R37.2
- new net 5V0: C43.1, J7.1
- new net TEMP_SENSE_EXT: R37.1

Commit message: JST headers fixed, no more errors, fully routed
Parts:
- J7: value Header_100mil_1x03 -> JST_PH_2.0mm_1x03; footprint sldrnrd:Header_100mil_1x03 -> sldrnrd:JST_PH_2.0mm_1x03; symbol sldrnrd:Connector/100Mil/Header_100mil_1x03 -> sldrnrd:Connector/JST/JST_PH_2.0mm_1x03; LCSC C225478 -> C131339; MPN A2541WV-3P -> B3B-PH-K-S; Manufacturer CJT -> JST
- R27, R29, R32, R33, R35, R36: symbol sldrnrd:Resistor/R_0603 -> sldrnrd:Resistor/R0603_5k1; LCSC (none) -> C23186; MPN (none) -> 0603WAF5101T5E; Manufacturer (none) -> Uni-Royal
- R28, R31: symbol sldrnrd:Resistor/R_0603 -> sldrnrd:Resistor/R0603_100k; LCSC (none) -> C25803; MPN (none) -> 0603WAF1003T5E; Manufacturer (none) -> Uni-Royal
- renumbered C41 to C38, C37 to C39, C38 to C40, C39 to C41, C40 to C42
